Commit message: feat: Add CycloneDDS configuration and update launch files for unified TF tree
- Created a new CycloneDDS profile XML configuration file for domain settings.
- Updated the bringup launch file to include a GroupAction for remapping TF topics to a unified namespace.
- Integrated TF relay nodes to connect external TF sources to the unified /leeloo namespace.
- Modified the Kinect TF computation node to use a dynamic robot base frame parameter.
- Added a new URDF file for the static structure connecting the Ridgeback and Doosan arm.
- Removed camera-related links from the main URDF as their poses are now managed dynamically.
- Updated package.xml to include dependencies for robot_state_publisher and topic_tools.
- Adjusted the Docker startup script to use a new image tag for the container.
- Commented out unnecessary repository entries in my.repos for clarity.

File: leeloo/urdf/leeloo.urdf (robot description, URDF)
Before this commit: robot ridgeback, 37 links, 36 joints
Links:
- removed link camera_base
- removed link camera_body
- removed link camera_visor
Joints:
- removed joint camera_base_to_body
- removed joint camera_base_to_visor
- removed joint camera_joint

Commit message: fix: Rename URDF links to match published TF frames and update comments for clarity

File: leeloo/urdf/leeloo.urdf (robot description, URDF)
Before this commit: robot ridgeback, 34 links, 33 joints
Links:
- removed link base_0
- removed link link1
- removed link link2
- removed link link3
- removed link link4
- removed link link5
- removed link link6
- removed link mid_mount
- added link default_mount
- added link dsr01/base_link, mass 4.12; collision mesh filename=package://leeloo/meshes/m1013_collision/MF1013_0_0.dae scale=0.001 0.001 0.001; visual mesh filename=package://leeloo/meshes/m1013_blue/MF1013_0_0.dae scale=0.001 0.001 0.001
- added link dsr01/link_1, mass 7.8; collision mesh filename=package://leeloo/meshes/m1013_collision/MF1013_1_0.dae scale=0.001 0.001 0.001; visual mesh filename=package://leeloo/meshes/m1013_blue/MF1013_1_0.dae scale=0.001 0.001 0.001
- added link dsr01/link_2, mass 10.83; collision mesh filename=package://leeloo/meshes/m1013_collision/MF1013_2_0.dae scale=0.001 0.001 0.001; collision mesh filename=package://leeloo/meshes/m1013_collision/MF1013_2_1.dae scale=0.001 0.001 0.001
- added link dsr01/link_3, mass 3.68; collision mesh filename=package://leeloo/meshes/m1013_collision/MF1013_3_0.dae scale=0.001 0.001 0.001; visual mesh filename=package://leeloo/meshes/m1013_blue/MF1013_3_0.dae scale=0.001 0.001 0.001
- added link dsr01/link_4, mass 3.82; collision mesh filename=package://leeloo/meshes/m1013_collision/MF1013_4_0.dae scale=0.001 0.001 0.001; collision mesh filename=package://leeloo/meshes/m1013_collision/MF1013_4_1.dae scale=0.001 0.001 0.001
- added link dsr01/link_5, mass 2.82; collision mesh filename=package://leeloo/meshes/m1013_collision/MF1013_5_0.dae scale=0.001 0.001 0.001; visual mesh filename=package://leeloo/meshes/m1013_blue/MF1013_5_0.dae scale=0.001 0.001 0.001
- added link dsr01/link_6, mass 1.16; collision mesh filename=package://leeloo/meshes/m1013_collision/MF1013_6_0.dae scale=0.001 0.001 0.001; visual mesh filename=package://leeloo/meshes/m1013_blue/MF1013_6_0.dae scale=0.001 0.001 0.001
- added link dsr01/world
Joints:
- added joint dsr01_base_link_joint: type fixed, parent dsr01/world, child dsr01/base_link, origin xyz=0 0 0 rpy=0 0 0
- joint arm_mount_joint: child base_0 -> dsr01/world
- joint joint1: child link1 -> dsr01/link_1; parent base_0 -> dsr01/base_link
- joint joint2: child link2 -> dsr01/link_2; parent link1 -> dsr01/link_1
- joint joint3: child link3 -> dsr01/link_3; parent link2 -> dsr01/link_2
- joint joint4: child link4 -> dsr01/link_4; parent link3 -> dsr01/link_3
- joint joint5: child link5 -> dsr01/link_5; parent link4 -> dsr01/link_4
- joint joint6: child link6 -> dsr01/link_6; parent link5 -> dsr01/link_5
- joint mid_mount_joint: child mid_mount -> default_mount
- joint structure_base_joint: parent mid_mount -> default_mount

Commit message: feat: Update ExecuteTrajectoryNode timer and message timing; add RidgebackTwist node for cmd_vel handling; modify voxel_map_publisher subscriptions; add Robotiq 2F-85 gripper to URDF

File: leeloo/urdf/leeloo.urdf (robot description, URDF)
Before this commit: robot ridgeback, 35 links, 34 joints
Links:
- added link robotiq_85_base_link, mass 0.636951; collision mesh filename=package://leeloo/meshes/collision/robotiq_85_base_link.stl; visual mesh filename=package://leeloo/meshes/visual/robotiq_85_base_link.dae
- added link robotiq_85_left_finger_link, mass 0.027309; collision mesh filename=package://leeloo/meshes/collision/robotiq_85_finger_link.stl; visual mesh filename=package://leeloo/meshes/visual/robotiq_85_finger_link.dae
- added link robotiq_85_left_finger_tip_link, mass 0.019555; collision mesh filename=package://leeloo/meshes/collision/robotiq_85_finger_tip_lin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; visual mesh filename=package://leeloo/meshes/visual/robotiq_85_finger_tip_link.d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
- added link robotiq_85_left_inner_knuckle_link, mass 0.029951; collision mesh filename=package://leeloo/meshes/collision/robotiq_85_inner_knuckle_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; visual mesh filename=package://leeloo/meshes/visual/robotiq_85_inner_knuckle_lin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
- added link robotiq_85_left_knuckle_link, mass 0.018491; collision mesh filename=package://leeloo/meshes/collision/robotiq_85_knuckle_link.s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; visual mesh filename=package://leeloo/meshes/visual/robotiq_85_knuckle_link.dae
- added link robotiq_85_right_finger_link, mass 0.027309; collision mesh filename=package://leeloo/meshes/collision/robotiq_85_finger_link.stl; visual mesh filename=package://leeloo/meshes/visual/robotiq_85_finger_link.dae
- added link robotiq_85_right_finger_tip_link, mass 0.019555; collision mesh filename=package://leeloo/meshes/collision/robotiq_85_finger_tip_lin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; visual mesh filename=package://leeloo/meshes/visual/robotiq_85_finger_tip_link.d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
- added link robotiq_85_right_inner_knuckle_link, mass 0.029951; collision mesh filename=package://leeloo/meshes/collision/robotiq_85_inner_knuckle_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; visual mesh filename=package://leeloo/meshes/visual/robotiq_85_inner_knuckle_lin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
- added link robotiq_85_right_knuckle_link, mass 0.018491; collision mesh filename=package://leeloo/meshes/collision/robotiq_85_knuckle_link.s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; visual mesh filename=package://leeloo/meshes/visual/robotiq_85_knuckle_link.dae
Joints:
- added joint robotiq_85_base_joint: type fixed, parent dsr01/link_6, child robotiq_85_base_link, origin xyz=0.0 0 0.0 rpy=0 -1.57 0
- added joint robotiq_85_left_finger_joint: type fixed, parent robotiq_85_left_knuckle_link, child robotiq_85_left_finger_link, origin xyz=-0.00408552455 -0.03148604435 0.0 rpy=0 0 0
- added joint robotiq_85_left_finger_tip_joint: type continuous, parent robotiq_85_left_inner_knuckle_link, child robotiq_85_left_finger_tip_link, origin xyz=0.04303959807 -0.03759940821 0.0 rpy=0.0 0.0 0.0, axis 0 0 1, limit lower=-3.14 upper=3.14 effort=0.1 velocity=100.0, mimic joint=robotiq_85_left_knuckle_joint multiplier=-1
- added joint robotiq_85_left_inner_knuckle_joint: type continuous, parent robotiq_85_base_link, child robotiq_85_left_inner_knuckle_link, origin xyz=0.06142 0.0127 0 rpy=3.141592653589793 0.0 0.0, axis 0 0 1, limit lower=-3.14 upper=3.14 effort=0.1 velocity=100.0, mimic joint=robotiq_85_left_knuckle_joint offset=0
- added joint robotiq_85_left_knuckle_joint: type revolute, parent robotiq_85_base_link, child robotiq_85_left_knuckle_link, origin xyz=0.05490451627 0.03060114443 0.0 rpy=3.141592653589793 0.0 0.0, axis 0 0 1, limit lower=0.0 upper=0.804 effort=50 velocity=0.5
- added joint robotiq_85_right_finger_joint: type fixed, parent robotiq_85_right_knuckle_link, child robotiq_85_right_finger_link, origin xyz=-0.00408552455 -0.03148604435 0.0 rpy=0 0 0
- added joint robotiq_85_right_finger_tip_joint: type continuous, parent robotiq_85_right_inner_knuckle_link, child robotiq_85_right_finger_tip_link, origin xyz=0.04303959807 -0.03759940821 0.0 rpy=0.0 0.0 0.0, axis 0 0 1, limit lower=-3.14 upper=3.14 effort=0.1 velocity=100.0, mimic joint=robotiq_85_left_knuckle_joint multiplier=-1
- added joint robotiq_85_right_inner_knuckle_joint: type continuous, parent robotiq_85_base_link, child robotiq_85_right_inner_knuckle_link, origin xyz=0.06142 -0.0127 0 rpy=0 0 0, axis 0 0 1, limit lower=-3.14 upper=3.14 effort=0.1 velocity=100.0, mimic joint=robotiq_85_left_knuckle_joint offset=0
- added joint robotiq_85_right_knuckle_joint: type continuous, parent robotiq_85_base_link, child robotiq_85_right_knuckle_link, origin xyz=0.05490451627 -0.03060114443 0.0 rpy=0.0 0.0 0.0, axis 0 0 1, limit lower=-3.14 upper=3.14 effort=50 velocity=100.0, mimic joint=robotiq_85_left_knuckle_joint

Commit message: feat: Enhance pose generation and saving functionality
- Updated pose_generator_node.py to use package share directory for default output path and improved goal execution handling.
- Enhanced pose_saver_node.py with new services for trajectory generation and execution, added goto_pose service to drive to saved poses, and improved redundancy checks.
- Introduced recalibrate_from_samples.py script for offline recalibration from saved samples, filtering points by ambiguity ratio and recalculating calibration using OpenCV.
- Updated package.xml to include new dependencies and added GotoPose service definition in leeloo_msgs.
- Modified CMakeLists.txt and setup.py to ensure proper installation of new service and launch files.

File: leeloo/urdf/leeloo.urdf (robot description, URDF)
Before this commit: robot ridgeback, 44 links, 43 joints
Links:
- link robotiq_85_base_link: mass 0.636951 -> 6.6320197e-01; geometry collision mesh filename=package://robotiq_description/meshes/collision/2f_85/roboti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; visual mesh filename=package://robotiq_description/meshes/visual/2f_85/robotiq_b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
- link robotiq_85_left_finger_link: mass 0.027309 -> 4.260376752e-02; geometry collision mesh filename=package://robotiq_description/meshes/collision/2f_85/left_f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; visual mesh filename=package://robotiq_description/meshes/visual/2f_85/left_fing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
- link robotiq_85_left_finger_tip_link: mass 0.019555 -> 4.268588744e-02; geometry collision mesh filename=package://robotiq_description/meshes/collision/2f_85/left_f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; visual mesh filename=package://robotiq_description/meshes/visual/2f_85/left_fing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
- link robotiq_85_left_inner_knuckle_link: mass 0.029951 -> 2.969376448e-02; geometry collision mesh filename=package://robotiq_description/meshes/collision/2f_85/left_i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; visual mesh filename=package://robotiq_description/meshes/visual/2f_85/left_inne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
- link robotiq_85_left_knuckle_link: mass 0.018491 -> 1.384773208e-02; geometry collision mesh filename=package://robotiq_description/meshes/collision/2f_85/left_k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; visual mesh filename=package://robotiq_description/meshes/visual/2f_85/left_knuc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
- link robotiq_85_right_finger_link: mass 0.027309 -> 4.260376752000000e-02; geometry collision mesh filename=package://robotiq_description/meshes/collision/2f_85/right_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; visual mesh filename=package://robotiq_description/meshes/visual/2f_85/right_fin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
- link robotiq_85_right_finger_tip_link: mass 0.019555 -> 4.268588744e-02; geometry collision mesh filename=package://robotiq_description/meshes/collision/2f_85/right_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; visual mesh filename=package://robotiq_description/meshes/visual/2f_85/right_fin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
- link robotiq_85_right_inner_knuckle_link: mass 0.029951 -> 2.969376448e-02; geometry collision mesh filename=package://robotiq_description/meshes/collision/2f_85/right_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; visual mesh filename=package://robotiq_description/meshes/visual/2f_85/right_inn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
- link robotiq_85_right_knuckle_link: mass 0.018491 -> 1.384773208e-02; geometry collision mesh filename=package://robotiq_description/meshes/collision/2f_85/right_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; visual mesh filename=package://robotiq_description/meshes/visual/2f_85/right_knu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
Joints:
- joint joint2: limit lower=-6.2832 upper=6.2832 effort=346 velocity=2.0944 -> lower=-2.0944 upper=2.0944 effort=346 velocity=2.0944
- joint joint3: limit lower=-2.35619 upper=2.35619 effort=163 velocity=3.1416 -> lower=-2.61799 upper=2.61799 effort=163 velocity=3.1416
- joint robotiq_85_base_joint: origin xyz=0.0 0 0.0 rpy=0 -1.57 0 -> xyz=0.0 0 0.0 rpy=0 0 1.5707963267948966
- joint robotiq_85_left_finger_joint: origin xyz=-0.00408552455 -0.03148604435 0.0 rpy=0 0 0 -> xyz=0.03152616 0.0 -0.00376347 rpy=0 0 0
- joint robotiq_85_left_finger_tip_joint: axis 0 0 1 -> 0 -1 0; limit lower=-3.14 upper=3.14 effort=0.1 velocity=100.0 -> lower=-0.8 upper=0.0 effort=50 velocity=0.5; origin xyz=0.04303959807 -0.03759940821 0.0 rpy=0.0 0.0 0.0 -> xyz=0.00563134 0.0 0.04718515 rpy=0 0 0; parent robotiq_85_left_inner_knuckle_link -> robotiq_85_left_finger_link; type continuous -> revolute
- joint robotiq_85_left_inner_knuckle_joint: axis 0 0 1 -> 0 -1 0; limit lower=-3.14 upper=3.14 effort=0.1 velocity=100.0 -> lower=0.0 upper=0.8 effort=50 velocity=0.5; mimic joint=robotiq_85_left_knuckle_joint offset=0 -> joint=robotiq_85_left_knuckle_joint; origin xyz=0.06142 0.0127 0 rpy=3.141592653589793 0.0 0.0 -> xyz=0.0127 0.0 0.06142 rpy=0 0 0; type continuous -> revolute
- joint robotiq_85_left_knuckle_joint: axis 0 0 1 -> 0 -1 0; limit lower=0.0 upper=0.804 effort=50 velocity=0.5 -> lower=0.0 upper=0.8 effort=50 velocity=0.5; origin xyz=0.05490451627 0.03060114443 0.0 rpy=3.141592653589793 0.0 0.0 -> xyz=0.03060114 0.0 0.05490452 rpy=0 0 0
- joint robotiq_85_right_finger_joint: origin xyz=-0.00408552455 -0.03148604435 0.0 rpy=0 0 0 -> xyz=-0.03152616 0.0 -0.00376347 rpy=0 0 0
- joint robotiq_85_right_finger_tip_joint: axis 0 0 1 -> 0 -1 0; limit lower=-3.14 upper=3.14 effort=0.1 velocity=100.0 -> lower=0.0 upper=0.8 effort=50 velocity=0.5; mimic joint=robotiq_85_left_knuckle_joint multiplier=-1 -> joint=robotiq_85_left_knuckle_joint; origin xyz=0.04303959807 -0.03759940821 0.0 rpy=0.0 0.0 0.0 -> xyz=-0.00563134 0.0 0.04718515 rpy=0 0 0; parent robotiq_85_right_inner_knuckle_link -> robotiq_85_right_finger_link; type continuous -> revolute
- joint robotiq_85_right_inner_knuckle_joint: axis 0 0 1 -> 0 -1 0; limit lower=-3.14 upper=3.14 effort=0.1 velocity=100.0 -> lower=-0.8 upper=0.0 effort=50 velocity=0.5; mimic joint=robotiq_85_left_knuckle_joint offset=0 -> joint=robotiq_85_left_knuckle_joint multiplier=-1; origin xyz=0.06142 -0.0127 0 rpy=0 0 0 -> xyz=-0.0127 0.0 0.06142 rpy=0 0 0; type continuous -> revolute
- joint robotiq_85_right_knuckle_joint: axis 0 0 1 -> 0 -1 0; limit lower=-3.14 upper=3.14 effort=50 velocity=100.0 -> lower=-0.8 upper=0.0 effort=50 velocity=0.5; mimic joint=robotiq_85_left_knuckle_joint -> joint=robotiq_85_left_knuckle_joint multiplier=-1; origin xyz=0.05490451627 -0.03060114443 0.0 rpy=0.0 0.0 0.0 -> xyz=-0.03060114 0.0 0.05490452 rpy=0 0 0; type continuous -> revolute
